File: powerprobe/powerprobe.kicad_sch (KiCad schematic)
At the start: 41 parts, among them SW3 OS103011MS8QP1, U1 LT3045EMSE-PBF, U2 OPA847xD, U3 LT3045EMSE-PBF, U4 LT3094EMSE-TRPBF

Commit message: Board finished
Connections:
- net 5V: now also U3.10 (OUTS), U3.12 (OUT)
- net V_TARGET: now also U1.10 (OUTS), U1.12 (OUT)
Changed lines of the file:
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@@
+	)
+	(junction
+		(at 233.68 33.02)
+		(diameter 0)
+		(color 0 0 0 0)
 	)
 	(junction
@@
 	)
 	(junction
+		(at 113.03 33.02)
+		(diameter 0)
+		(color 0 0 0 0)
+	)
+	(junction
 		(at 241.3 50.8)
 		(diameter 0)
@@
 	(wire
 		(pts
+			(xy 233.68 33.02) (xy 233.68 35.56)
+		)
+		(stroke
+			(width 0)
+			(type default)
+		)
+	)
+	(wire
+		(pts
 			(xy 179.07 33.02) (xy 179.07 30.48)
 		)
@@
 	(wire
 		(pts
+			(xy 233.68 30.48) (xy 233.68 33.02)
+		)
+		(stroke
+			(width 0)
+			(type default)
+		)
+	)
+	(wire
+		(pts
 			(xy 140.97 85.09) (xy 140.97 87.63)
 		)
@@
 	(wire
 		(pts
-			(xy 99.06 33.02) (xy 129.54 33.02)
+			(xy 99.06 33.02) (xy 113.03 33.02)
 		)
 		(stroke
@@
 	(wire
 		(pts
+			(xy 233.68 33.02) (xy 250.19 33.02)
+		)
+		(stroke
+			(width 0)
+			(type default)
+		)
+	)
+	(wire
+		(pts
 			(xy 102.87 118.11) (xy 102.87 120.65)
 		)
@@
 	(wire
 		(pts
-			(xy 233.68 30.48) (xy 233.68 35.56)
-		)
-		(stroke
-			(width 0)
-			(type default)
-		)
-	)
-	(wire
-		(pts
 			(xy 175.26 44.45) (xy 175.26 40.64)
 		)
@@
 	(wire
 		(pts
+			(xy 219.71 30.48) (xy 233.68 30.48)
+		)
+		(stroke
+			(width 0)
+			(type default)
+		)
+	)
+	(wire
+		(pts
+			(xy 113.03 33.02) (xy 113.03 35.56)
+		)
+		(stroke
+			(width 0)
+			(type default)
+		)
+	)
+	(wire
+		(pts
 			(xy 102.87 46.99) (xy 111.76 46.99)
 		)
@@
 	(wire
 		(pts
+			(xy 113.03 33.02) (xy 129.54 33.02)
+		)
+		(stroke
+			(width 0)
+			(type default)
+		)
+	)
+	(wire
+		(pts
 			(xy 214.63 134.62) (xy 226.06 134.62)
 		)
@@
 	(wire
 		(pts
-			(xy 219.71 33.02) (xy 250.19 33.02)
+			(xy 219.71 33.02) (xy 233.68 33.02)
 		)
 		(stroke
@@
 	(wire
 		(pts
-			(xy 113.03 30.48) (xy 113.03 35.56)
-		)
-		(stroke
-			(width 0)
-			(type default)
-		)
-	)
-	(wire
-		(pts
 			(xy 261.62 27.94) (xy 261.62 50.8)
 		)
@@
 	(wire
 		(pts
-			(xy 219.71 30.48) (xy 233.68 30.48)
-		)
-		(stroke
+			(xy 113.03 30.48) (xy 113.03 33.02)
+		)
+		(stroke
