File: powerprobe/powerprobe.kicad_pcb (KiCad board)
At the start: 2 copper layers, 41 parts, among them SW3 OS103011MS8QP1, U1 LT3045EMSE-PBF, U2 OPA847xD, U3 LT3045EMSE-PBF, U4 LT3094EMSE-TRPBF

Commit message: Some more routing
Parts:
- moved R10 5.33 mm to (167.8, 82.5)
- moved H3 1.15 mm to (191.0, 100.5)
- moved C10 1.11 mm to (165.7, 82.6)
- moved H2 1.10 mm to (191.9, 73.0)
- moved SW3 1.03 mm to (151.5, 74.5)
- moved FB2 0.89 mm to (172.1, 83.5)
- moved C8 0.81 mm to (149.6, 96.6)
- moved R7 0.69 mm to (153.4, 96.7)
- moved C7 0.66 mm to (155.2, 91.8)
- moved U1 0.54 mm to (151.0, 91.5)
- moved C13 0.53 mm to (171.9, 74.6)
- moved U3 0.41 mm to (161.8, 85.9)
- moved U4 0.30 mm to (176.8, 74.6)
- moved C11 0.23 mm to (161.7, 80.3)
- moved C9 0.20 mm to (160.6, 91.0)
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Routing:
- net 5V: track 0.00 -> 16.2 mm, vias 0 -> 2
- net /V_BAT+: track 0.00 -> 13.3 mm, vias 0 -> 2
- net GND: track 5.92 -> 12.4 mm
- net Net-(U3-SET): track 0.00 -> 6.46 mm
- net Net-(U3-ILIM): track 0.00 -> 2.91 mm
- net Net-(U4-ILIM): track 2.74 -> 0.03 mm
- net /V_BAT-: track 7.12 -> 8.87 mm
- net Net-(U2-V+): track 14.6 -> 13.8 mm

Commit message: Board finished
Parts:
- moved J_BAT2 23.1 mm to (164.5, 72.8), turned to 180 degrees
- moved J_BAT1 22.0 mm to (146.9, 72.8), turned to 0 degrees
- moved SW3 16.6 mm to (143.9, 89.3), turned to 180 degrees
- moved C6 11.6 mm to (158.2, 92.6), turned to 90 degrees
- moved C9 8.64 mm to (158.1, 82.7), turned to 90 degrees
- moved C7 8.37 mm to (151.2, 84.5), turned to 180 degrees
- moved R9 7.77 mm to (158.0, 86.5), turned to 90 degrees
- moved J_TARGET1 6.50 mm to (163.0, 92.8)
- moved C11 5.27 mm to (166.9, 79.4), turned to 0 degrees
- moved H4 4.27 mm to (138.4, 97.2)
- moved C10 3.61 mm to (167.6, 85.7)
- moved R10 3.61 mm to (169.7, 85.6)
- moved FB1 3.53 mm to (182.9, 76.7), turned to 180 degrees
- moved H3 3.41 mm to (191.8, 97.2)
- moved H1 3.13 mm to (138.4, 73.2)
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Connections:
- U1 pad 10: Net-(U1-OUTS) -> V_TARGET
- U1 pad 12: Net-(U1-OUTS) -> V_TARGET
- U3 pad 10: Net-(U3-OUTS) -> 5V
- U3 pad 12: Net-(U3-OUTS) -> 5V
Routing:
- net GND: track 12.4 -> 172.4 mm, vias 0 -> 10
- net /V_BAT+: track 13.3 -> 58.4 mm
- net /R_VT: track 0.00 -> 19.7 mm
- net V_TARGET: track 0.00 -> 18.1 mm, vias 0 -> 1
- net /V_BAT-: track 8.87 -> 16.4 mm
- net /R_3V3: track 0.00 -> 7.33 mm
- net /R_1V2: track 0.00 -> 6.69 mm
- net /R_1V8: track 0.00 -> 6.69 mm
- net 5V: track 16.2 -> 9.56 mm, vias 2 -> 0
- net -5V: track 11.3 -> 6.68 mm
- net Net-(U2-V-): track 16.5 -> 20.7 mm
- net Net-(U1-ILIM): track 0.00 -> 3.45 mm
- net Net-(U4-ILIM): track 0.03 -> 2.89 mm
- net Net-(U3-SET): track 6.46 -> 4.45 mm
- net VSS_TARGET: track 14.0 -> 12.2 mm
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- added copper zone on B.Cu, net GND
Other:
- board outline added: 63.4 x 34 mm
- board text added: "1.2V"
- board text added: "1.8V"
- board text added: "3.3V"

Commit message: Add gerber files
Other:
- board text added: "powerprobe rev1.0 Carles Pey"
Changed lines of the file:
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@@
 			(outputformat 1)
 			(mirror no)
-			(drillshape 1)
+			(drillshape 0)
 			(scaleselection 1)
-			(outputdirectory "")
+			(outputdirectory "gerbers/")
 		)
 	)
@@
 			)
 			(justify left bottom)
+		)
+	)
+	(gr_text "powerprobe rev1.0\nCarles Pey"
+		(at 171.6 97.35 0)
+		(layer "F.SilkS")
+		(effects
+			(font
+				(size 1 1)
+				(thickness 0.125)
+				(italic yes)
+			)
+			(justify left bottom)
